Commit message: feat(nav): add SLAM stack (EKF, scan_angle_fixer, slam_toolbox, saved map)
New cargo_bot_navigation (ekf.yaml, slam_toolbox.yaml, maps/cuarto_v1) and cargo_bot_bringup (scan_angle_fixer, slam/localization launches); imu_link upgrade in sensors.xacro; regenerated Isaac URDF; RViz SLAM config.

Co-Authored-By: Claude Opus 4.8 <noreply@anthropic.com>

File: src/cargo_bot_description/urdf/sensors.xacro (robot description, xacro)
@@ -32,5 +32,7 @@
         <origin xyz="0 0 0" rpy="0 0 0"/>
     </sensor>
-    <link name="imu_link"/>
+    <link name="imu_link">
+          <xacro:inertial_box mass="0.01" x="0.02" y="0.02" z="0.005"/>
+      </link>
     <joint name="imu_joint" type="fixed">
         <parent link="base_link"/>
@@ -38,3 +40,7 @@
         <origin xyz="0 0 0" rpy="0 0 0"/>
     </joint>
+    <sensor name="imu" type="imu" update_rate="100">
+        <parent link="imu_link"/>
+        <origin xyz="0 0 0" rpy="0 0 0"/>
+    </sensor>
 </robot>
