Commit message: chore: corregir paths hardcodeados tras mover workspace a Documentos\
El workspace se movio de C:\Users\agusp\cargo_bot_ws (y su espejo WSL
/mnt/c/Users/agusp/cargo_bot_ws) a la carpeta Documentos\. Docs, scripts
.cmd/.sh y utilidades de diagnostico Python seguian referenciando la
ubicacion vieja.

File: cargo_bot_isaac.urdf (robot description, URDF)
Before this commit: robot cargo_bot, 7 links, 6 joints
Links:
- link base_link: geometry collision mesh filename=C:/Users/agusp/Documentos/cargo_bot_ws/src/cargo_bot_descri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 scale=0.001 0.001 0.001; visual mesh filename=C:/Users/agusp/Documentos/cargo_bot_ws/src/cargo_bot_descri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 scale=0.001 0.001 0.001
- link caster_wheel_link: geometry collision mesh filename=C:/Users/agusp/Documentos/cargo_bot_ws/src/cargo_bot_descri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 scale=0.001 0.001 0.001; visual mesh filename=C:/Users/agusp/Documentos/cargo_bot_ws/src/cargo_bot_descri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 scale=0.001 0.001 0.001
- link left_wheel_link: geometry collision mesh filename=C:/Users/agusp/Documentos/cargo_bot_ws/src/cargo_bot_descri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 scale=0.001 0.001 0.001; visual mesh filename=C:/Users/agusp/Documentos/cargo_bot_ws/src/cargo_bot_descri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 scale=0.001 0.001 0.001
- link lidar_link: geometry collision mesh filename=C:/Users/agusp/Documentos/cargo_bot_ws/src/cargo_bot_descri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 scale=0.001 0.001 0.001; visual mesh filename=C:/Users/agusp/Documentos/cargo_bot_ws/src/cargo_bot_descri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 scale=0.001 0.001 0.001
- link right_wheel_link: geometry collision mesh filename=C:/Users/agusp/Documentos/cargo_bot_ws/src/cargo_bot_descri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 scale=0.001 0.001 0.001; visual mesh filename=C:/Users/agusp/Documentos/cargo_bot_ws/src/cargo_bot_descri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 scale=0.001 0.001 0.001

File: src/cargo_bot_description/urdf/cargo_bot_isaac.urdf (robot description, URDF)
Before this commit: robot cargo_bot, 7 links, 6 joints
Links:
- link base_link: geometry collision mesh filename=/mnt/c/Users/agusp/Documentos/cargo_bot_ws/src/cargo_bot_de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 scale=0.001 0.001 0.001; visual mesh filename=/mnt/c/Users/agusp/Documentos/cargo_bot_ws/src/cargo_bot_de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 scale=0.001 0.001 0.001
- link caster_wheel_link: geometry collision mesh filename=/mnt/c/Users/agusp/Documentos/cargo_bot_ws/src/cargo_bot_de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 scale=0.001 0.001 0.001; visual mesh filename=/mnt/c/Users/agusp/Documentos/cargo_bot_ws/src/cargo_bot_de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 scale=0.001 0.001 0.001
- link left_wheel_link: geometry collision mesh filename=/mnt/c/Users/agusp/Documentos/cargo_bot_ws/src/cargo_bot_de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 scale=0.001 0.001 0.001; visual mesh filename=/mnt/c/Users/agusp/Documentos/cargo_bot_ws/src/cargo_bot_de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 scale=0.001 0.001 0.001
- link lidar_link: geometry collision mesh filename=/mnt/c/Users/agusp/Documentos/cargo_bot_ws/src/cargo_bot_de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 scale=0.001 0.001 0.001; visual mesh filename=/mnt/c/Users/agusp/Documentos/cargo_bot_ws/src/cargo_bot_de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 scale=0.001 0.001 0.001
- link right_wheel_link: geometry collision mesh filename=/mnt/c/Users/agusp/Documentos/cargo_bot_ws/src/cargo_bot_de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 scale=0.001 0.001 0.001; visual mesh filename=/mnt/c/Users/agusp/Documentos/cargo_bot_ws/src/cargo_bot_de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 scale=0.001 0.001 0.001
